Commit message: Add Robotiq 3 Finger Gripper
Added Robotiq 3 Finger Gripper to URDF and updated SRDF to acommodate.

File: ceccrebot_demo_support/urdf/ur10_robot.urdf.xacro (robot description, xacro)
@@ -7,3 +7,11 @@
   <!-- arm -->
   <xacro:ur10_robot prefix="ur_" joint_limited="false"/>
+  <!-- Robotiq Gripper -->
+  <xacro:include filename="$(find robotiq_s_model_visualization)/cfg/s-model_mesh_macro.xacro" />
+  <xacro:s-model_mesh  prefix=""/>
+  <joint name="EEjoint" type ="fixed">
+    <origin rpy="0 0 0" xyz="0 0 0.160"/>
+    <parent link="ur_tool0"/>
+    <child link="palm"/>
+  </joint>
 </robot>
