Commit message: Small edits for getting robot online in demo workcell

File: ceccrebot_demo_support/urdf/environment_macros.xacro (robot description, xacro)
@@ -9,5 +9,5 @@
       <link name="${root_frame_id}"/>
       <!-- Robot support -->
-      <xacro:platform name="cnc" parent_link="${root_frame_id}" thickness="${platform_thickness}" material="orange">
+      <xacro:platform name="cnc" parent_link="${root_frame_id}" length="0.1" width="0.1" height="${platform_thickness}" material="orange">
         <origin xyz="0.0 0.0 ${platform_thickness}"/>
       </xacro:platform>

File: ceccrebot_demo_support/urdf/hardware_macros.xacro (robot description, xacro)
@@ -2,10 +2,10 @@
 <robot xmlns:xacro="http://ros.org/wiki/xacro">
   <!-- Robot support -->
-  <xacro:macro name="platform" params="name parent_link thickness material *location">
+  <xacro:macro name="platform" params="name parent_link length width height material *location">
     <link name="${name}_platform_link">
       <visual>
-        <origin xyz="0.0 0.0 -${thickness * 0.5}" rpy="0 0 0"/>
-        <geometry>
-          <box size="0.5 0.5 ${thickness}"/>
+        <origin xyz="0.0 0.0 -${height * 0.5}" rpy="0 0 0"/>
+        <geometry>
+          <box size="${length} ${width} ${height}"/>
         </geometry>
         <material name="${material}"/>
@@ -13,7 +13,7 @@
       <collision name="{name}_platform">
         <geometry>
-          <box size="0.6 0.6 ${thickness}"/>
-        </geometry>
-        <origin xyz="0.0 0.0 -${thickness * 0.5}" rpy="0 0 0"/>
+          <box size="${length} ${width} ${height}"/>
+        </geometry>
+        <origin xyz="0.0 0.0 -${height * 0.5}" rpy="0 0 0"/>
       </collision>
     </link>
@@ -66,4 +66,7 @@
   <!-- VM5i CNC -->
   <xacro:macro name="cnc_VM5i" params="id parent_link *location">
+    <!-- Machine reference point in STL -->
+    <!-- x = right, y = up, z = out front door -->
+    <!-- x = -50.0, y = 1054.28, z = 207.0 -->
     <link name="cnc_${id}_base">
       <visual>

File: ceccrebot_demo_support/urdf/ur10_robot.urdf.xacro (robot description, xacro)
@@ -15,3 +15,10 @@
     <child link="palm"/>
   </joint>
+  <!-- TCP (2018-07-17) -->
+  <link name="ur_center_grip_tcp"/>
+  <joint name="ur_center_grip_tcp_joint" type="fixed">
+    <origin xyz="0 0 0.187" rpy="0 0 0"/>
+    <parent link="ur_tool0"/>
+    <child link="ur_center_grip_tcp"/>
+  </joint>
 </robot>

Commit message: Add table to environment

File: ceccrebot_demo_support/urdf/environment_macros.xacro (robot description, xacro)
@@ -7,8 +7,13 @@
       <!-- parameters -->
       <xacro:property name="platform_thickness" value="1.0414"/>
+      <xacro:property name="table_height" value="1.0541"/>
       <link name="${root_frame_id}"/>
       <!-- Robot support -->
       <xacro:platform name="cnc" parent_link="${root_frame_id}" length="0.1" width="0.1" height="${platform_thickness}" material="orange">
         <origin xyz="0.0 0.0 ${platform_thickness}"/>
+      </xacro:platform>
+      <!-- Part table -->
+      <xacro:platform name="part_table" parent_link="${root_frame_id}" length="0.9144" width="0.762" height="${table_height}" material="light_gray">
+          <origin xyz="0.6858 0.4572 ${table_height}" rpy="0 0 1.5708"/>
       </xacro:platform>
       <!-- CNC -->
