Commit message: Consolidate single robot demo environment

File: ceccrebot_demo_support/urdf/ur10_in_scene.urdf.xacro (robot description, xacro)
@@ -1,10 +1,40 @@
 <?xml version="1.0"?>
 <robot xmlns:xacro="http://ros.org/wiki/xacro" name="ur10">
-  <!-- common stuff -->
+  <xacro:include filename="$(find ceccrebot_demo_support)/urdf/hardware_macros.xacro" />
+  <xacro:include filename="$(find ceccrebot_demo_support)/urdf/materials.xacro"/>
   <xacro:include filename="$(find ur_description)/urdf/common.gazebo.xacro" />
-  <!-- ur10 -->
   <xacro:include filename="$(find ur_description)/urdf/ur10.urdf.xacro" />
-  <!-- arm -->
+  <xacro:property name="root_frame_id" value="world_frame"/>
+  <xacro:property name="platform_thickness" value="1.0414"/>
+  <xacro:property name="table_height" value="1.0541"/>
+  <!-- root link -->
+  <link name="${root_frame_id}"/>
+  <!-- Robot support -->
+  <xacro:platform name="robot" parent_link="${root_frame_id}" length="0.1" width="0.1" height="${platform_thickness}" material="orange">
+    <origin xyz="0.0 0.0 ${platform_thickness}"/>
+  </xacro:platform>
+  <!-- Part table -->
+  <xacro:platform name="part_table" parent_link="${root_frame_id}" length="0.9144" width="0.762" height="${table_height}" material="light_gray">
+      <origin xyz="-0.4572 0.6858 ${table_height}" rpy="0 0 0"/>
+  </xacro:platform>
+  <!-- CNC -->
+  <xacro:cnc_VM5i id="A" parent_link="${root_frame_id}">
+    <origin xyz="0.75 -0.5 0.0" rpy="0 0 3.1415"/>
+  </xacro:cnc_VM5i>
+  <!-- CMM -->
+  <xacro:cmm id="A" parent_link="${root_frame_id}">
+    <origin xyz="1.403 0.085 0.91" rpy="0 0 1.5708"/>
+  </xacro:cmm>
+  <!-- Demo Parts -->
+  <xacro:part id="1" parent_link="${root_frame_id}">
+    <origin xyz="0.75 0.5 0.95 " rpy="0 0 -1.5708"/>
+  </xacro:part>
+  <!-- Robot -->
   <xacro:ur10_robot prefix="ur_" joint_limited="false"/>
+  <joint name="robot_platform_to_robot_joint" type="fixed">
+    <origin xyz="0 0 0" rpy="0 0 0.1"/>
+    <parent link="robot_platform_link"/>
+    <child link="ur_base_link"/>
+  </joint>
   <!-- Robotiq Gripper -->
   <xacro:include filename="$(find robotiq_s_model_visualization)/cfg/s-model_mesh_macro.xacro" />
@@ -15,11 +45,3 @@
     <child link="palm"/>
   </joint>
-  <!-- environment -->
-  <xacro:include filename="$(find ceccrebot_demo_support)/urdf/environment_macros.xacro" />
-  <xacro:single_robot_demo_env root_frame_id="env_frame"/>
-  <joint name="environment_jt" type ="fixed">
-    <origin rpy="0 0 0" xyz="0 0 -1.0414"/>
-    <parent link="ur_base_link"/>
-    <child link="env_frame"/>
-  </joint>
 </robot>

Commit message: Update the gripper URDF for better visuals

File: ceccrebot_demo_support/urdf/ur10_in_scene.urdf.xacro (robot description, xacro)
@@ -40,8 +40,8 @@
   </joint>
   <!-- Robotiq Gripper -->
-  <xacro:include filename="$(find robotiq_s_model_visualization)/cfg/s-model_mesh_macro.xacro" />
-  <xacro:s-model_mesh  prefix=""/>
+  <xacro:include filename="$(find robotiq_s_model_visualization)/cfg/s-model_articulated_macro.xacro" />
+  <xacro:s-model_articulated prefix=""/>
   <joint name="EEjoint" type ="fixed">
-    <origin rpy="0 0 -0.4" xyz="0 0 0.160"/>
+    <origin rpy="1.571 0 -0.4" xyz="0 0 0.04"/>
     <parent link="ur_tool0"/>
     <child link="palm"/>

Commit message: Update the gripper URDF for better visuals

File: ceccrebot_demo_support/urdf/ur10_in_scene.urdf.xacro (robot description, xacro)
@@ -38,8 +38,8 @@
   </joint>
   <!-- Robotiq Gripper -->
-  <xacro:include filename="$(find robotiq_s_model_visualization)/cfg/s-model_mesh_macro.xacro" />
-  <xacro:s-model_mesh  prefix=""/>
+  <xacro:include filename="$(find robotiq_s_model_visualization)/cfg/s-model_articulated_macro.xacro" />
+  <xacro:s-model_articulated prefix=""/>
   <joint name="EEjoint" type ="fixed">
-    <origin rpy="0 0 0" xyz="0 0 0.160"/>
+    <origin rpy="1.571 0 0" xyz="0 0 0.04"/>
     <parent link="ur_tool0"/>
     <child link="palm"/>

Commit message: Working demo as of Friday night

File: ceccrebot_demo_support/urdf/ur10_in_scene.urdf.xacro (robot description, xacro)
@@ -7,5 +7,5 @@
   <xacro:property name="root_frame_id" value="world_frame"/>
   <xacro:property name="platform_thickness" value="1.0414"/>
-  <xacro:property name="table_height" value="1.045"/>
+  <xacro:property name="table_height" value="1.01"/>
   <!-- root link -->
   <link name="${root_frame_id}"/>
@@ -15,19 +15,21 @@
   </xacro:platform>
   <!-- Part table -->
-  <xacro:platform name="part_table" parent_link="${root_frame_id}" length="0.9144" width="0.762" height="${table_height}" material="light_gray">
-      <origin xyz="-0.525 0.69 ${table_height}" rpy="0 0 0"/>
+  <xacro:platform name="part_table" parent_link="${root_frame_id}" length="1.016" width="0.610" height="${table_height}" material="light_gray">
+      <origin xyz="-0.345 0.788	 ${table_height}" rpy="0 0 0"/>
   </xacro:platform>
   <!-- CNC -->
   <xacro:cnc_VM5i id="A" parent_link="${root_frame_id}">
-    <origin xyz="0.75 -0.5 0.0" rpy="0 0 3.1415"/>
+    <origin xyz="0.60 -0.55 0.0" rpy="0 0 3.1415"/>
   </xacro:cnc_VM5i>
   <!-- CMM -->
   <xacro:cmm id="A" parent_link="${root_frame_id}">
-    <origin xyz="1.49 0.07 0.83" rpy="0 0 1.5708"/>
+    <origin xyz="1.68 0.15 0.815" rpy="0 0 1.5708"/>
   </xacro:cmm>
   <!-- Demo Parts -->
+  <!--
   <xacro:part id="1" parent_link="${root_frame_id}">
     <origin xyz="0.75 0.5 0.95 " rpy="0 0 -1.5708"/>
   </xacro:part>
+  -->
   <!-- Robot -->
   <xacro:ur10_robot prefix="ur_" joint_limited="true" elbow_joint_lower_limit="-2.6"/>
@@ -41,5 +43,5 @@
   <xacro:s-model_mesh  prefix=""/>
   <joint name="EEjoint" type ="fixed">
-    <origin rpy="0 0 0" xyz="0 0 0.160"/>
+    <origin rpy="0 0 -0.4" xyz="0 0 0.160"/>
     <parent link="ur_tool0"/>
     <child link="palm"/>

Commit message: Bring in fixed-joint version of articulated Robotiq S Model

File: ceccrebot_demo_support/urdf/ur10_in_scene.urdf.xacro (robot description, xacro)
@@ -39,10 +39,26 @@
     <child link="ur_base_link"/>
   </joint>
+  <link name="ur_gripper_adapter_link">
+    <visual>
+      <origin xyz="0 0 -0.015"/>
+      <geometry>
+          <cylinder radius="0.04" length="0.03"/>
+      </geometry>
+      <material name="darkblue">
+        <color rgba="0.4 0.4 1 1"/>
+      </material>
+    </visual>
+  </link>
+  <joint name="gripper_adapter_joint" type="fixed">
+    <origin xyz="0 0 0.03" rpy="0 0 0"/>
+    <parent link="ur_tool0"/>
+    <child link="ur_gripper_adapter_link"/>
+  </joint>
   <!-- Robotiq Gripper -->
-  <xacro:include filename="$(find robotiq_s_model_visualization)/cfg/s-model_articulated_macro.xacro" />
+  <xacro:include filename="$(find ceccrebot_demo_support)/urdf/robotiq/s-model_articulated_macro.xacro" />
   <xacro:s-model_articulated prefix=""/>
   <joint name="EEjoint" type ="fixed">
     <origin rpy="1.571 0 -0.4" xyz="0 0 0.04"/>
-    <parent link="ur_tool0"/>
+    <parent link="ur_gripper_adapter_link"/>
     <child link="palm"/>
   </joint>

Commit message: Bring in fixed-joint version of articulated Robotiq S Model

File: ceccrebot_demo_support/urdf/ur10_in_scene.urdf.xacro (robot description, xacro)
@@ -37,10 +37,26 @@
     <child link="ur_base_link"/>
   </joint>
+  <link name="ur_gripper_adapter_link">
+    <visual>
+      <origin xyz="0 0 -0.015"/>
+      <geometry>
+          <cylinder radius="0.04" length="0.03"/>
+      </geometry>
+      <material name="darkblue">
+        <color rgba="0.4 0.4 1 1"/>
+      </material>
+    </visual>
+  </link>
+  <joint name="gripper_adapter_joint" type="fixed">
+    <origin xyz="0 0 0.03" rpy="0 0 0"/>
+    <parent link="ur_tool0"/>
+    <child link="ur_gripper_adapter_link"/>
+  </joint>
   <!-- Robotiq Gripper -->
-  <xacro:include filename="$(find robotiq_s_model_visualization)/cfg/s-model_articulated_macro.xacro" />
+  <xacro:include filename="$(find ceccrebot_demo_support)/urdf/robotiq/s-model_articulated_macro.xacro" />
   <xacro:s-model_articulated prefix=""/>
   <joint name="EEjoint" type ="fixed">
     <origin rpy="1.571 0 0" xyz="0 0 0.04"/>
-    <parent link="ur_tool0"/>
+    <parent link="ur_gripper_adapter_link"/>
     <child link="palm"/>
   </joint>
