Commit message: Change CMM to Hexagon
Added Hexagon stl to meshes folder and modified the URDFs with the new collision layer and offsets.

File: ceccrebot_demo_support/urdf/hardware_macros.xacro (robot description, xacro)
@@ -63,5 +63,5 @@
       <visual>
         <geometry>
-          <mesh filename="package://ceccrebot_demo_support/meshes/CMM_color.dae"/>
+          <mesh filename="package://ceccrebot_demo_support/meshes/Hexagon-MI-TIGOSF-CADModelwHP-S-X1.stl" scale = "0.001 0.001 0.001" />
         </geometry>
         <material name="light_gray"/>
@@ -69,25 +69,31 @@
       <collision name="cmm_${id}_base">
         <geometry>
-          <box size="2.2 1.3 1.0"/>
+          <box size=".8 1.25 0.95"/>
         </geometry>
-        <origin xyz="0.0 -0.65 0.5"/>
+        <origin xyz="0.3 0.6 -.4"/>
       </collision>
       <collision name="cmm_${id}_probe_area">
         <geometry>
-          <box size="1.2 0.5 1.2"/>
+          <box size=".25 .25 1.3"/>
         </geometry>
-        <origin xyz="0.5 -0.4 2.15"/>
+        <origin xyz="0.35 0.675 0.95"/>
       </collision>
-      <collision name="cmm_${id}_right_wall">
+      <collision name="cmm_${id}_back_wall">
         <geometry>
-          <box size="0.4 1.5 1.0"/>
+          <box size="1.25 0.5 1.0"/>
         </geometry>
-        <origin xyz="1.0 -0.7 1.5"/>
+        <origin xyz=".5 .2 0.5"/>
       </collision>
-      <collision name="cmm_${id}_left_wall">
+      <collision name="cmm_${id}_probe_gantry">
         <geometry>
-          <box size="0.3 0.4 1.0"/>
+          <box size="0.35 1.4 0.25"/>
         </geometry>
-        <origin xyz="-0.2 -0.4 1.5"/>
+        <origin xyz="0.4 0.475 0.75"/>
+      </collision>
+      <collision name="cmm_${id}_computer">
+        <geometry>
+          <box size="0.5 0.5 1.0"/>
+        </geometry>
+        <origin xyz="-0.5 0.9 0.1"/>
       </collision>
     </link>

File: ceccrebot_demo_support/urdf/multi_robot_demo_env.xacro (robot description, xacro)
@@ -36,5 +36,5 @@
   <!-- CMM -->
   <xacro:cmm id="A" parent_link="${root_frame_id}">
-    <origin xyz="-2.5 2.5 0.0" />
+    <origin xyz="-1.5 2.0 0.85" rpy="0 0 3.1415"/>
   </xacro:cmm>
   <xacro:conveyor id="1" parent_link="${root_frame_id}">

File: ceccrebot_demo_support/urdf/single_robot_demo_env.xacro (robot description, xacro)
@@ -25,5 +25,5 @@
   <!-- CMM -->
   <xacro:cmm id="A" parent_link="${root_frame_id}">
-    <origin xyz="0.5 -2.5 0.0" rpy="0 0 3.1415"/>
+    <origin xyz="-0.5 -2.2 0.85" rpy="0 0 0"/>
   </xacro:cmm>
   <xacro:conveyor id="1" parent_link="${root_frame_id}">

Commit message: Add Demo Part. Remove Conveyor
Added demo part to the environment as a static part and remove the conveyors.

File: ceccrebot_demo_support/urdf/hardware_macros.xacro (robot description, xacro)
@@ -126,3 +126,25 @@
     </joint>
   </xacro:macro>
+  <!-- Demo Part-->
+  <xacro:macro name="part" params="id parent_link *location">
+    <link name="part_${id}">
+      <visual>
+        <geometry>
+          <mesh filename="package://ceccrebot_demo_support/meshes/AMTDemoPart.stl" scale = "0.001 0.001 0.001"/>
+        </geometry>
+        <origin xyz="0 0 0.0" rpy="0 0 0"/>
+      </visual>
+      <collision name="part_${id}_coll">
+        <geometry>
+          <box size="0.1 0.2 0.3"/>
+        </geometry>
+        <origin xyz="0.0 0.0 0.0"/>
+      </collision>
+    </link>
+    <joint name="part_${id}" type ="fixed">
+      <xacro:insert_block name="location" />
+      <parent link="${parent_link}"/>
+      <child link="part_${id}"/>
+    </joint>
+  </xacro:macro>
 </robot>

File: ceccrebot_demo_support/urdf/single_robot_demo_env.xacro (robot description, xacro)
@@ -27,15 +27,7 @@
     <origin xyz="-0.5 -2.2 0.85" rpy="0 0 0"/>
   </xacro:cmm>
-  <xacro:conveyor id="1" parent_link="${root_frame_id}">
-    <origin xyz="1.75 0.0 0.0" />
-  </xacro:conveyor>
-  <xacro:conveyor id="2" parent_link="${root_frame_id}">
-    <origin xyz="3.25 0.0 0.0" />
-  </xacro:conveyor>
-  <xacro:conveyor id="3" parent_link="${root_frame_id}">
-    <origin xyz="-1.75 0.0 0.0" />
-  </xacro:conveyor>
-  <xacro:conveyor id="4" parent_link="${root_frame_id}">
-    <origin xyz="-3.25 0.0 0.0" />
-  </xacro:conveyor>
+  <!-- Demo Parts -->
+  <xacro:part id="1" parent_link="${root_frame_id}">
+    <origin xyz="0 -1.25 0.95 " rpy="0 0 0"/>
+  </xacro:part>
 </robot>

Commit message: Replace CNC with Hurco VM5i
Added Hurco VM5i to URDF file and replaced the CNC in the single robot demo.

File: ceccrebot_demo_support/urdf/hardware_macros.xacro (robot description, xacro)
@@ -50,4 +50,51 @@
         </geometry>
         <origin xyz="1.625 0.8 1.45"/>
+      </collision>
+    </link>
+    <joint name="cnc_${id}_joint" type ="fixed">
+      <xacro:insert_block name="location" />
+      <parent link="${parent_link}"/>
+      <child link="cnc_${id}_base"/>
+    </joint>
+  </xacro:macro>
+  <!-- VM5i CNC -->
+  <xacro:macro name="cnc_VM5i" params="id parent_link *location">
+    <link name="cnc_${id}_base">
+      <visual>
+        <origin xyz="0.0 1.75 0.0" rpy="1.571 0 0"/>
+        <geometry>
+          <mesh filename="package://ceccrebot_demo_support/meshes/VM5i.stl" scale = "0.001 0.001 0.001"/>
+        </geometry>
+        <material name="light_gray"/>
+      </visual>
+      <collision name="cnc_${id}_base">
+        <geometry>
+          <box size="1.6 1.8 0.8"/>
+        </geometry>
+        <origin xyz="0.8 0.9 0.4" />
+      </collision>
+      <collision name="cnc_${id}_back">
+        <geometry>
+          <box size="1.60 1.25 2.0"/>
+        </geometry>
+        <origin xyz="0.8 1.05 1.0" />
+      </collision>
+      <collision name="cnc_${id}_right_wall">
+        <geometry>
+          <box size="0.65 1.7 2.0"/>
+        </geometry>
+        <origin xyz="1.32 0.85 1.0" />
+      </collision>
+      <collision name="cnc_${id}_left_wall">
+        <geometry>
+          <box size="0.4 1.7 2.0"/>
+        </geometry>
+        <origin xyz="0.2 0.85 1.0" />
+      </collision>
+      <collision name="cnc_${id}_computer">
+        <geometry>
+          <box size="0.5 1.2 0.8"/>
+        </geometry>
+        <origin xyz="1.4 -0.6 1.5"/>
       </collision>
     </link>

File: ceccrebot_demo_support/urdf/single_robot_demo_env.xacro (robot description, xacro)
@@ -15,19 +15,19 @@
   <joint name="platform_to_base_joint" type ="fixed">
     <origin xyz="0 0 0" rpy="0 0 0"/>
-    <parent link="robot_platform_link"/>
+    <parent link="robot_platform_link"/
     <child link="cnc_robot_base_link"/>
   </joint>
   -->
   <!-- CNC -->
-  <xacro:cnc id="A" parent_link="${root_frame_id}">
-    <origin xyz="1.0 2.7 0.0" rpy="0 0 3.1415"/>
-  </xacro:cnc>
+  <xacro:cnc_VM5i id="A" parent_link="${root_frame_id}">
+    <origin xyz="-0.75 -0.5 0.0" rpy="0 0 1.571"/>
+  </xacro:cnc_VM5i>
   <!-- CMM -->
   <xacro:cmm id="A" parent_link="${root_frame_id}">
-    <origin xyz="-0.5 -2.2 0.85" rpy="0 0 0"/>
+    <origin xyz="0.0 -1.75 0.85" rpy="0 0 0"/>
   </xacro:cmm>
   <!-- Demo Parts -->
   <xacro:part id="1" parent_link="${root_frame_id}">
-    <origin xyz="0 -1.25 0.95 " rpy="0 0 0"/>
+    <origin xyz="0.5 -0.75 0.95 " rpy="0 0 0"/>
   </xacro:part>
 </robot>

Commit message: Change VM5i to mesh with doors open

File: ceccrebot_demo_support/urdf/hardware_macros.xacro (robot description, xacro)
@@ -64,5 +64,5 @@
         <origin xyz="0.0 1.75 0.0" rpy="1.571 0 0"/>
         <geometry>
-          <mesh filename="package://ceccrebot_demo_support/meshes/VM5i.stl" scale = "0.001 0.001 0.001"/>
+          <mesh filename="package://ceccrebot_demo_support/meshes/VM5i_DoorsOpen.stl" scale = "0.001 0.001 0.001"/>
         </geometry>
         <material name="light_gray"/>

Commit message: Change stand height to 42"

File: ceccrebot_demo_support/urdf/hardware_macros.xacro (robot description, xacro)
@@ -11,4 +11,10 @@
         <material name="${material}"/>
       </visual>
+      <collision name="{name}_platform">
+        <geometry>
+          <box size="0.6 0.6 ${thickness}"/>
+        </geometry>
+        <origin xyz="0.0 0.0 -${thickness * 0.5}" rpy="0 0 0"/>
+      </collision>
     </link>
     <joint name="${name}_platform_joint" type ="fixed">

File: ceccrebot_demo_support/urdf/multi_robot_demo_env.xacro (robot description, xacro)
@@ -5,5 +5,5 @@
   <xacro:include filename="$(find ceccrebot_demo_support)/urdf/materials.xacro"/>
   <!-- parameters -->
-  <xacro:property name="platform_thickness" value="0.5"/>
+  <xacro:property name="platform_thickness" value="1.0414"/>
   <xacro:property name="root_frame_id" value="world_frame"/>
   <link name="${root_frame_id}"/>

File: ceccrebot_demo_support/urdf/single_robot_demo_env.xacro (robot description, xacro)
@@ -5,5 +5,5 @@
   <xacro:include filename="$(find ceccrebot_demo_support)/urdf/materials.xacro"/>
   <!-- parameters -->
-  <xacro:property name="platform_thickness" value="0.5"/>
+  <xacro:property name="platform_thickness" value="1.0414"/>
   <xacro:property name="root_frame_id" value="world_frame"/>
   <link name="${root_frame_id}"/>

Commit message: Lighter meshes for hardware

File: ceccrebot_demo_support/urdf/hardware_macros.xacro (robot description, xacro)
@@ -73,5 +73,5 @@
         <origin xyz="0.0 1.75 0.0" rpy="1.571 0 0"/>
         <geometry>
-          <mesh filename="package://ceccrebot_demo_support/meshes/VM5i_DoorsOpen.stl" scale = "0.001 0.001 0.001"/>
+          <mesh filename="package://ceccrebot_demo_support/meshes/VM5i_DoorsOpen_lightweight.stl" scale = "0.001 0.001 0.001"/>
         </geometry>
         <material name="light_gray"/>
@@ -119,5 +119,5 @@
       <visual>
         <geometry>
-          <mesh filename="package://ceccrebot_demo_support/meshes/Hexagon-MI-TIGOSF-CADModelwHP-S-X1.stl" scale = "0.001 0.001 0.001" />
+          <mesh filename="package://ceccrebot_demo_support/meshes/Hexagon-MI-TIGOSF-CADModelwHP-S-X1_lightweight.stl" scale = "0.001 0.001 0.001" />
         </geometry>
         <material name="light_gray"/>

Commit message: Dump of integration work at Hurco

File: ceccrebot_demo_support/urdf/hardware_macros.xacro (robot description, xacro)
@@ -85,5 +85,5 @@
       <collision name="cnc_${id}_back">
         <geometry>
-          <box size="1.60 1.25 2.0"/>
+          <box size="1.60 0.75 2.0"/>
         </geometry>
         <origin xyz="0.8 1.05 1.0" />
@@ -101,4 +101,5 @@
         <origin xyz="0.2 0.85 1.0" />
       </collision>
+      <!--
       <collision name="cnc_${id}_computer">
         <geometry>
@@ -107,4 +108,5 @@
         <origin xyz="1.4 -0.6 1.5"/>
       </collision>
+      -->
     </link>
     <joint name="cnc_${id}_joint" type ="fixed">

File: ceccrebot_demo_support/urdf/ur10_in_scene.urdf.xacro (robot description, xacro)
@@ -7,5 +7,5 @@
   <xacro:property name="root_frame_id" value="world_frame"/>
   <xacro:property name="platform_thickness" value="1.0414"/>
-  <xacro:property name="table_height" value="1.0541"/>
+  <xacro:property name="table_height" value="1.045"/>
   <!-- root link -->
   <link name="${root_frame_id}"/>
@@ -16,5 +16,5 @@
   <!-- Part table -->
   <xacro:platform name="part_table" parent_link="${root_frame_id}" length="0.9144" width="0.762" height="${table_height}" material="light_gray">
-      <origin xyz="-0.4572 0.6858 ${table_height}" rpy="0 0 0"/>
+      <origin xyz="-0.525 0.69 ${table_height}" rpy="0 0 0"/>
   </xacro:platform>
   <!-- CNC -->
@@ -24,5 +24,5 @@
   <!-- CMM -->
   <xacro:cmm id="A" parent_link="${root_frame_id}">
-    <origin xyz="1.403 0.085 0.91" rpy="0 0 1.5708"/>
+    <origin xyz="1.49 0.07 0.83" rpy="0 0 1.5708"/>
   </xacro:cmm>
   <!-- Demo Parts -->
@@ -31,7 +31,7 @@
   </xacro:part>
   <!-- Robot -->
-  <xacro:ur10_robot prefix="ur_" joint_limited="false"/>
+  <xacro:ur10_robot prefix="ur_" joint_limited="true" elbow_joint_lower_limit="-2.6"/>
   <joint name="robot_platform_to_robot_joint" type="fixed">
-    <origin xyz="0 0 0" rpy="0 0 0.1"/>
+    <origin xyz="0 0 0" rpy="0 0 0.02"/>
     <parent link="robot_platform_link"/>
     <child link="ur_base_link"/>

Commit message: Update Hexagon URDF
Move the gantry position in the collision model to match where it is in the stowed position

File: ceccrebot_demo_support/urdf/hardware_macros.xacro (robot description, xacro)
@@ -135,5 +135,5 @@
           <box size=".25 .25 1.3"/>
         </geometry>
-        <origin xyz="0.35 0.675 0.95"/>
+        <origin xyz="0.55 0.675 0.95"/>
       </collision>
       <collision name="cmm_${id}_back_wall">
@@ -147,5 +147,5 @@
           <box size="0.35 1.4 0.25"/>
         </geometry>
-        <origin xyz="0.4 0.475 0.75"/>
+        <origin xyz="0.6 0.475 0.75"/>
       </collision>
       <collision name="cmm_${id}_computer">

Commit message: Update Collision geometry for tool change
This greatly reduced (probably too far), but it is necessary to reach the back right corner where the tool change currently is.

File: ceccrebot_demo_support/urdf/hardware_macros.xacro (robot description, xacro)
@@ -81,9 +81,9 @@
           <box size="1.6 1.8 0.8"/>
         </geometry>
-        <origin xyz="0.8 0.9 0.4" />
+        <origin xyz="0.8 0.9 0.3" />
       </collision>
       <collision name="cnc_${id}_back">
         <geometry>
-          <box size="1.60 0.75 2.0"/>
+          <box size="1.40 0.35 2.0"/>
         </geometry>
         <origin xyz="0.8 1.05 1.0" />
@@ -91,7 +91,7 @@
       <collision name="cnc_${id}_right_wall">
         <geometry>
-          <box size="0.65 1.7 2.0"/>
-        </geometry>
-        <origin xyz="1.32 0.85 1.0" />
+          <box size="0.15 1.7 2.0"/>
+        </geometry>
+        <origin xyz="1.42 0.85 1.0" />
       </collision>
       <collision name="cnc_${id}_left_wall">

Commit message: Model of table at IMTS demo

File: ceccrebot_demo_support/urdf/hardware_macros.xacro (robot description, xacro)
@@ -11,4 +11,98 @@
         <material name="${material}"/>
       </visual>
+      <collision name="{name}_platform">
+        <geometry>
+          <box size="${length} ${width} ${height}"/>
+        </geometry>
+        <origin xyz="0.0 0.0 -${height * 0.5}" rpy="0 0 0"/>
+      </collision>
+    </link>
+    <joint name="${name}_platform_joint" type ="fixed">
+      <xacro:insert_block name="location"/>
+      <parent link="${parent_link}"/>
+      <child link="${name}_platform_link"/>
+    </joint>
+  </xacro:macro>
+  <xacro:macro name="part_table" params="name parent_link length width height *location">
+    <link name="${name}_platform_link">
+      <!-- Main blue body -->
+      <visual>
+        <origin xyz="0.0 0.0 -0.457" rpy="0 0 0"/>
+        <geometry>
+          <box size="0.635 0.457 0.711"/>
+        </geometry>
+        <material name="teal_blue"/>
+      </visual>
+      <!-- Left gray panel -->
+      <visual>
+        <origin xyz="-0.3365 0.0 -0.546" rpy="0 0 0"/>
+        <geometry>
+          <box size="0.038 0.508 0.940"/>
+        </geometry>
+        <material name="light_gray">
+            <color rgba="0.8 0.8 0.8 0.1"/>
+        </material>
+      </visual>
+      <!-- Right gray panel -->
+      <visual>
+        <origin xyz="0.3365 0.0 -0.546" rpy="0 0 0"/>
+        <geometry>
+          <box size="0.038 0.508 0.940"/>
+        </geometry>
+        <material name="light_gray">
+            <color rgba="0.8 0.8 0.8 0.1"/>
+        </material>
+      </visual>
+      <!-- Glass surface -->
+      <visual>
+        <origin xyz="0.0 -0.05 -0.006" rpy="0 0 0"/>
+        <geometry>
+          <box size="1.016 0.610 0.012"/>
+        </geometry>
+        <material name="glass">
+            <color rgba="0.8 0.8 0.8 0.1"/>
+        </material>
+      </visual>
+      <!-- Front left steel post -->
+      <visual>
+        <origin xyz="-0.3365 -0.16 -0.0444" rpy="0 0 0"/>
+        <geometry>
+          <cylinder length="0.064" radius="0.013"/>
+        </geometry>
+        <material name="steel">
+            <color rgba="0.8 0.8 0.8 0.1"/>
+        </material>
+      </visual>
+      <!-- Front right steel post -->
+      <visual>
+        <origin xyz="0.3365 -0.16 -0.0444" rpy="0 0 0"/>
+        <geometry>
+          <cylinder length="0.064" radius="0.013"/>
+        </geometry>
+        <material name="steel">
+            <color rgba="0.8 0.8 0.8 0.1"/>
+        </material>
+      </visual>
+      <!-- Back left steel post -->
+      <visual>
+        <origin xyz="-0.3365 0.16 -0.0444" rpy="0 0 0"/>
+        <geometry>
+          <cylinder length="0.064" radius="0.013"/>
+        </geometry>
+        <material name="steel">
+            <color rgba="0.8 0.8 0.8 0.1"/>
+        </material>
+      </visual>
+      <!-- Back right steel post -->
+      <visual>
+        <origin xyz="0.3365 0.16 -0.0444" rpy="0 0 0"/>
+        <geometry>
+          <cylinder length="0.064" radius="0.013"/>
+        </geometry>
+        <material name="steel">
+            <color rgba="0.8 0.8 0.8 0.1"/>
+        </material>
+      </visual>
+      <!-- One unified collision geometry -->
       <collision name="{name}_platform">
         <geometry>

File: ceccrebot_demo_support/urdf/materials.xacro (robot description, xacro)
@@ -16,4 +16,7 @@
     <color rgba="0.78 0.94 0.965 1"/>
   </material>
+  <material name="teal_blue">
+    <color rgba="0.0 0.7 0.96 1"/>
+  </material>
   <material name="light_gray">
     <color rgba="0.7 0.7 0.7 1"/>

File: ceccrebot_demo_support/urdf/ur10_in_scene.urdf.xacro (robot description, xacro)
@@ -1,6 +1,6 @@
 <?xml version="1.0"?>
 <robot xmlns:xacro="http://ros.org/wiki/xacro" name="ur10">
+  <xacro:include filename="$(find ceccrebot_demo_support)/urdf/materials.xacro"/>
   <xacro:include filename="$(find ceccrebot_demo_support)/urdf/hardware_macros.xacro" />
-  <xacro:include filename="$(find ceccrebot_demo_support)/urdf/materials.xacro"/>
   <xacro:include filename="$(find ur_description)/urdf/common.gazebo.xacro" />
   <xacro:include filename="$(find ur_description)/urdf/ur10.urdf.xacro" />
@@ -15,7 +15,7 @@
   </xacro:platform>
   <!-- Part table -->
-  <xacro:platform name="part_table" parent_link="${root_frame_id}" length="1.016" width="0.610" height="${table_height}" material="light_gray">
+  <xacro:part_table name="part_table" parent_link="${root_frame_id}" length="1.016" width="0.610" height="${table_height}">
       <origin xyz="-0.345 0.788	 ${table_height}" rpy="0 0 0"/>
-  </xacro:platform>
+  </xacro:part_table>
   <!-- CNC -->
   <xacro:cnc_VM5i id="A" parent_link="${root_frame_id}">
